File: Hardware/Controller.brd (EAGLE design)
At the start: 40 x 26 mm, 12 parts

Commit message: removed extra i2c resistors
Parts:
- removed R2, R3: (no value), rcl:R1206
Connections:
- net I2CCLK: no longer R3.1
- net I2CSDA: no longer R2.1
- net VCC: no longer R2.2, R3.2
Routing:
- net VCC: track 69.4 -> 56.6 mm, vias 5 -> 3
- net I2CCLK: track 24.7 -> 22.8 mm
- net I2CSDA: track 23.8 -> 22.6 mm
Changed lines of the file:
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@@
 <attribute name="VALUE" x="9.16" y="7.31" size="1.27" layer="27"/>
-</element>
-<element name="R2" library="rcl" library_urn="urn:adsk.eagle:library:334" package="R1206" package3d_urn="urn:adsk.eagle:package:23540/2" value="" x="10.13" y="18.27" smashed="yes">
-<attribute name="NAME" x="8.86" y="19.54" size="1.27" layer="25"/>
-<attribute name="POPULARITY" value="19" x="10.13" y="18.27" size="1.778" layer="27" display="off"/>
-<attribute name="SPICEPREFIX" value="R" x="10.13" y="18.27" size="1.778" layer="27" display="off"/>
-<attribute name="VALUE" x="8.86" y="15.73" size="1.27" layer="27"/>
-</element>
-<element name="R3" library="rcl" library_urn="urn:adsk.eagle:library:334" package="R1206" package3d_urn="urn:adsk.eagle:package:23540/2" value="" x="10.13" y="22.89" smashed="yes">
-<attribute name="NAME" x="8.86" y="24.16" size="1.27" layer="25"/>
-<attribute name="POPULARITY" value="19" x="10.13" y="22.89" size="1.778" layer="27" display="off"/>
-<attribute name="SPICEPREFIX" value="R" x="10.13" y="22.89" size="1.778" layer="27" display="off"/>
-<attribute name="VALUE" x="8.86" y="20.35" size="1.27" layer="27"/>
 </element>
 <element name="JP1" library="pinhead" library_urn="urn:adsk.eagle:library:325" package="1X01" package3d_urn="urn:adsk.eagle:package:22485/2" value="" x="36.48" y="4.01" smashed="yes">
@@
 <signal name="I2CSDA">
 <contactref element="U$1" pad="15"/>
-<contactref element="R2" pad="1"/>
 <contactref element="JP5" pad="1"/>
-<wire x1="4.35" y1="19.69" x2="7.288" y2="19.69" width="0.254" layer="1"/>
-<wire x1="7.288" y1="19.69" x2="8.708" y2="18.27" width="0.254" layer="1"/>
-<wire x1="8.708" y1="18.27" x2="11.088" y2="20.65" width="0.254" layer="1"/>
 <wire x1="16.85" y1="23.9" x2="22.875" y2="23.9" width="0.254" layer="1"/>
 <wire x1="22.875" y1="23.9" x2="22.875" y2="21.73" width="0.254" layer="1"/>
 <wire x1="22.875" y1="21.73" x2="22.775" y2="21.63" width="0.254" layer="1"/>
-<wire x1="11.088" y1="20.65" x2="13.6" y2="20.65" width="0.254" layer="1"/>
-<wire x1="13.6" y1="20.65" x2="16.85" y2="23.9" width="0.254" layer="1"/>
+<wire x1="12.64" y1="19.69" x2="16.85" y2="23.9" width="0.254" layer="1"/>
+<wire x1="4.35" y1="19.69" x2="12.64" y2="19.69" width="0.254" layer="1"/>
 </signal>
 <signal name="I2CCLK">
 <contactref element="U$1" pad="14"/>
-<contactref element="R3" pad="1"/>
 <contactref element="JP5" pad="2"/>
-<wire x1="4.35" y1="22.23" x2="8.048" y2="22.23" width="0.254" layer="1"/>
-<wire x1="8.048" y1="22.23" x2="8.708" y2="22.89" width="0.254" layer="1"/>
-<wire x1="8.708" y1="22.89" x2="8.708" y2="21.842" width="0.254" layer="1"/>
-<wire x1="8.708" y1="21.842" x2="9.2" y2="21.35" width="0.254" layer="1"/>
-<wire x1="9.2" y1="21.35" x2="13.4" y2="21.35" width="0.254" layer="1"/>
-<wire x1="13.4" y1="21.35" x2="16.5" y2="24.45" width="0.254" layer="1"/>
+<wire x1="4.35" y1="22.23" x2="7.95" y2="22.23" width="0.254" layer="1"/>
+<wire x1="8.048" y1="22.23" x2="7.95" y2="22.23" width="0.254" layer="1"/>
 <wire x1="16.5" y1="24.45" x2="23.4" y2="24.45" width="0.254" layer="1"/>
 <wire x1="23.4" y1="24.45" x2="23.425" y2="24.425" width="0.254" layer="1"/>
 <wire x1="23.425" y1="24.425" x2="23.425" y2="21.63" width="0.254" layer="1"/>
+<wire x1="8.048" y1="22.23" x2="14.28" y2="22.23" width="0.254" layer="1"/>
+<wire x1="14.28" y1="22.23" x2="16.5" y2="24.45" width="0.254" layer="1"/>
 </signal>
 <signal name="VCC">
 <contactref element="R1" pad="2"/>
 <contactref element="U$1" pad="1"/>
-<contactref element="R2" pad="2"/>
-<contactref element="R3" pad="2"/>
 <contactref element="JP1" pad="1"/>
 <contactref element="JP3" pad="2"/>
 <contactref element="U$2" pad="P$3"/>
 <contactref element="U$2" pad="P$2"/>
-<wire x1="11.552" y1="22.89" x2="11.862" y2="23.2" width="0.254" layer="1"/>
-<wire x1="11.862" y1="23.2" x2="13.65" y2="23.2" width="0.254" layer="1"/>
-<via x="13.65" y="23.2" extent="1-16" drill="0.55"/>
-<wire x1="13.65" y1="23.2" x2="13.65" y2="19.6" width="0.254" layer="16"/>
-<wire x1="13.65" y1="19.6" x2="13.65" y2="15.65" width="0.254" layer="16"/>
 <wire x1="13.65" y1="15.65" x2="13.65" y2="13.55" width="0.254" layer="16"/>
 <wire x1="13.65" y1="13.55" x2="13.5" y2="13.4" width="0.254" layer="16"/>
 <wire x1="13.5" y1="13.4" x2="9.715" y2="13.4" width="0.254" layer="16"/>
-<wire x1="13" y1="19.668" x2="11.602" y2="18.27" width="0.254" layer="1"/>
-<wire x1="11.552" y1="18.27" x2="11.602" y2="18.27" width="0.254" layer="1"/>
-<wire x1="13" y1="19.8" x2="12.95" y2="19.8" width="0.254" layer="1"/>
-<wire x1="13" y1="19.8" x2="13" y2="19.668" width="0.254" layer="1"/>
-<via x="12.95" y="19.8" extent="1-16" drill="0.55"/>
-<wire x1="13.65" y1="19.6" x2="13.15" y2="19.6" width="0.254" layer="16"/>
-<wire x1="13.15" y1="19.6" x2="12.95" y2="19.8" width="0.254" layer="16"/>
 <wire x1="11.852" y1="9.85" x2="13.052" y2="11.05" width="0.254" layer="1"/>
 <wire x1="13.052" y1="11.05" x2="13.45" y2="11.05" width="0.254" layer="1"/>

Commit message: cam jobs and battery updates for controller and speaker boards
Parts:
- moved U$2 3.92 mm to (22.1, 17.3)
Routing:
- net VCC: track 56.6 -> 90.1 mm
- net RST/SBWTDIO: track 29.2 -> 37.9 mm
- net TEST/SBWTCK: track 23.5 -> 24.0 mm
Other:
- outline, holes or cut-outs redrawn
- board text added: ":D"
Changed lines of the file:
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@@
 <plain>
 <wire x1="0" y1="0" x2="40" y2="0" width="0" layer="20"/>
-<wire x1="40" y1="0" x2="40.05" y2="25.95" width="0" layer="20"/>
-<wire x1="40.05" y1="25.95" x2="0" y2="26" width="0" layer="20"/>
+<wire x1="40" y1="0" x2="40" y2="26" width="0" layer="20"/>
+<wire x1="40" y1="26" x2="0" y2="26" width="0" layer="20"/>
 <wire x1="0" y1="26" x2="0" y2="0" width="0" layer="20"/>
 <text x="28.25" y="20.05" size="0.8128" layer="21">CLARG
@@
 <text x="1.9" y="20.9" size="0.4064" layer="21" rot="SR270">I2CSDA</text>
 <circle x="19.3" y="16.9" radius="0.26925625" width="0.1524" layer="21"/>
+<text x="38.2" y="11.65" size="0.8128" layer="21" rot="R180">:D</text>
 </plain>
 <attributes>
@@
 <attribute name="VALUE" x="7.98" y="0.965" size="1.27" layer="27"/>
 </element>
-<element name="U$2" library="Personal" package="3002BATTERY" value="3002BATTERY" x="22.54" y="13.4" smashed="yes" rot="MR0"/>
+<element name="U$2" library="Personal" package="3002BATTERY" value="3002BATTERY" x="22.14" y="17.3" smashed="yes" rot="MR0"/>
 <element name="CSUPPLY" library="rcl" library_urn="urn:adsk.eagle:library:334" package="C1206" package3d_urn="urn:adsk.eagle:package:23618/2" value="" x="16.6" y="13.85" smashed="yes">
 <attribute name="NAME" x="14.38" y="11.87" size="0.8128" layer="25"/>
@@
 <contactref element="U$1" pad="17"/>
 <contactref element="JP3" pad="4"/>
-<wire x1="4.61" y1="12.3" x2="9.06" y2="16.75" width="0.254" layer="1"/>
-<wire x1="9.06" y1="16.75" x2="12.45" y2="16.75" width="0.254" layer="1"/>
-<wire x1="12.45" y1="16.75" x2="14.05" y2="18.35" width="0.254" layer="1"/>
-<wire x1="17" y1="23.15" x2="20.65" y2="23.15" width="0.254" layer="1"/>
-<wire x1="20.65" y1="23.15" x2="21.475" y2="22.325" width="0.254" layer="1"/>
-<wire x1="21.475" y1="22.325" x2="21.475" y2="21.63" width="0.254" layer="1"/>
-<wire x1="14.05" y1="18.35" x2="14.05" y2="20.2" width="0.254" layer="1"/>
-<wire x1="14.05" y1="20.2" x2="17" y2="23.15" width="0.254" layer="1"/>
+<wire x1="21.475" y1="22.325" x2="21.475" y2="22.15" width="0.254" layer="1"/>
+<wire x1="21.475" y1="22.15" x2="21.475" y2="21.63" width="0.254" layer="1"/>
+<wire x1="4.61" y1="12.3" x2="4.61" y2="14.76" width="0.254" layer="1"/>
+<wire x1="17.6" y1="22.95" x2="21.45" y2="22.95" width="0.254" layer="1"/>
+<wire x1="21.45" y1="22.95" x2="21.475" y2="22.925" width="0.254" layer="1"/>
+<wire x1="21.475" y1="22.925" x2="21.475" y2="22.325" width="0.254" layer="1"/>
+<wire x1="4.61" y1="14.76" x2="8.15" y2="18.3" width="0.254" layer="1"/>
+<wire x1="8.15" y1="18.3" x2="12.95" y2="18.3" width="0.254" layer="1"/>
+<wire x1="12.95" y1="18.3" x2="17.6" y2="22.95" width="0.254" layer="1"/>
 </signal>
 <signal name="RST/SBWTDIO">
@@
 <wire x1="4.7" y1="9.85" x2="9.008" y2="9.85" width="0.254" layer="1"/>
 <wire x1="9.008" y1="9.85" x2="9.5" y2="10.342" width="0.254" layer="1"/>
-<wire x1="9.5" y1="10.342" x2="9.5" y2="15.6" width="0.254" layer="1"/>
-<wire x1="9.5" y1="15.6" x2="9.9" y2="16" width="0.254" layer="1"/>
-<wire x1="17.3" y1="20.25" x2="18.05" y2="20.25" width="0.254" layer="1"/>
-<via x="18.05" y="20.25" extent="1-16" drill="0.55"/>
-<wire x1="18.05" y1="20.25" x2="22.15" y2="20.25" width="0.254" layer="16"/>
-<wire x1="9.9" y1="16" x2="13.05" y2="16" width="0.254" layer="1"/>
-<wire x1="13.05" y1="16" x2="17.3" y2="20.25" width="0.254" layer="1"/>
-<wire x1="22.15" y1="20.25" x2="22.15" y2="22.8424" width="0.254" layer="16"/>
-<wire x1="22.15" y1="22.8424" x2="22" y2="22.9924" width="0.254" layer="16"/>
-<via x="22" y="22.9924" extent="1-16" drill="0.55"/>
-<wire x1="22" y1="22.9924" x2="22.125" y2="22.8674" width="0.254" layer="1"/>
-<wire x1="22.125" y1="22.8674" x2="22.125" y2="21.63" width="0.254" layer="1"/>
+<wire x1="9.008" y1="9.85" x2="9.008" y2="11.242" width="0.254" layer="1"/>
+<wire x1="9.008" y1="11.242" x2="5.8" y2="14.45" width="0.254" layer="1"/>
+<via x="5.8" y="14.45" extent="1-16" drill="0.508"/>
+<wire x1="5.8" y1="14.45" x2="3.55" y2="14.45" width="0.254" layer="16"/>
+<wire x1="3.55" y1="14.45" x2="3.35" y2="14.65" width="0.254" layer="16"/>
+<via x="3.35" y="14.65" extent="1-16" drill="0.508"/>
+<wire x1="3.35" y1="14.65" x2="7.75" y2="19.05" width="0.254" layer="1"/>
+<wire x1="17.3436" y1="23.4936" x2="22.1" y2="23.4936" width="0.254" layer="1"/>
+<wire x1="22.1" y1="23.4936" x2="22.125" y2="23.4686" width="0.254" layer="1"/>
+<wire x1="22.125" y1="23.4686" x2="22.125" y2="21.63" width="0.254" layer="1"/>
+<wire x1="7.75" y1="19.05" x2="12.9" y2="19.05" width="0.254" layer="1"/>
+<wire x1="12.9" y1="19.05" x2="17.3436" y2="23.4936" width="0.254" layer="1"/>
 </signal>
 <signal name="I2CSDA">
@@
 <contactref element="U$2" pad="P$3"/>
 <contactref element="U$2" pad="P$2"/>
-<wire x1="13.65" y1="15.65" x2="13.65" y2="13.55" width="0.254" layer="16"/>
-<wire x1="13.65" y1="13.55" x2="13.5" y2="13.4" width="0.254" layer="16"/>
-<wire x1="13.5" y1="13.4" x2="9.715" y2="13.4" width="0.254" layer="16"/>
-<wire x1="11.852" y1="9.85" x2="13.052" y2="11.05" width="0.254" layer="1"/>
-<wire x1="13.052" y1="11.05" x2="13.45" y2="11.05" width="0.254" layer="1"/>
-<via x="13.45" y="11.05" extent="1-16" drill="0.55"/>
-<wire x1="13.45" y1="11.05" x2="13.5" y2="11.1" width="0.254" layer="16"/>
-<wire x1="13.5" y1="11.1" x2="13.5" y2="13.4" width="0.254" layer="16"/>
-<wire x1="4.61" y1="7.22" x2="9.62" y2="7.22" width="0.254" layer="16"/>
-<wire x1="9.62" y1="7.22" x2="13.45" y2="11.05" width="0.254" layer="16"/>
-<wire x1="36.48" y1="4.01" x2="36.48" y2="12.285" width="0.254" layer="16"/>
-<wire x1="36.48" y1="12.285" x2="35.365" y2="13.4" width="0.254" layer="16"/>
+<wire x1="36.48" y1="4.01" x2="36.48" y2="15.785" width="0.254" layer="16"/>
+<wire x1="36.48" y1="15.785" x2="34.965" y2="17.3" width="0.254" layer="16"/>
 <wire x1="19.5251" y1="15.8299" x2="18.6799" y2="15.8299" width="0.254" layer="1"/>
 <wire x1="18.6799" y1="15.8299" x2="18.65" y2="15.8" width="0.254" layer="1"/>
-<via x="18.65" y="15.8" extent="1-16" drill="0.55"/>
-<wire x1="18.65" y1="15.8" x2="14.8" y2="15.8" width="0.254" layer="16"/>
-<wire x1="14.8" y1="15.8" x2="13.8" y2="15.8" width="0.254" layer="16"/>
-<wire x1="13.8" y1="15.8" x2="13.65" y2="15.65" width="0.254" layer="16"/>
-<wire x1="18.65" y1="15.8" x2="32.965" y2="15.8" width="0.1524" layer="16"/>
-<wire x1="32.965" y1="15.8" x2="35.365" y2="13.4" width="0.1524" layer="16"/>
+<wire x1="32.565" y1="19.7" x2="34.965" y2="17.3" width="0.1524" layer="16"/>
 <contactref element="CSUPPLY" pad="1"/>
-<wire x1="15.2" y1="13.85" x2="15.2" y2="15.4" width="0.1524" layer="1"/>
-<wire x1="15.2" y1="15.4" x2="14.8" y2="15.8" width="0.1524" layer="1"/>
-<via x="14.8" y="15.8" extent="1-16" drill="0.55"/>
+<wire x1="18.6799" y1="15.8299" x2="17.1799" y2="15.8299" width="0.254" layer="1"/>
+<wire x1="17.1799" y1="15.8299" x2="15.2" y2="13.85" width="0.254" layer="1"/>
+<wire x1="11.852" y1="9.85" x2="9.222" y2="7.22" width="0.254" layer="1"/>
+<wire x1="9.222" y1="7.22" x2="4.61" y2="7.22" width="0.254" layer="1"/>
+<wire x1="11.852" y1="9.85" x2="11.852" y2="10.502" width="0.254" layer="1"/>
+<wire x1="11.852" y1="10.502" x2="15.2" y2="13.85" width="0.254" layer="1"/>
+<wire x1="34.965" y1="17.3" x2="34.965" y2="25.2063625" width="0.254" layer="16"/>
+<wire x1="7.67169375" y1="25.206665625" x2="7.649909375" y2="25.22845" width="0.254" layer="1"/>
+<via x="7.649909375" y="25.22845" extent="1-16" drill="0.508"/>
+<wire x1="7.649909375" y1="25.22845" x2="7.649909375" y2="18.965090625" width="0.254" layer="16"/>
+<wire x1="7.649909375" y1="18.965090625" x2="9.315" y2="17.3" width="0.254" layer="16"/>
+<wire x1="9.315" y1="14.985" x2="9.315" y2="16.2" width="0.254" layer="16"/>
+<wire x1="9.315" y1="16.2" x2="9.315" y2="17.3" width="0.254" layer="16"/>
+<wire x1="7.649909375" y1="25.22845" x2="25.320828125" y2="25.22845" width="0.254" layer="1"/>
+<wire x1="25.320828125" y1="25.22845" x2="25.342915625" y2="25.2063625" width="0.254" layer="1"/>
+<wire x1="9" y1="12.702" x2="9" y2="13.8" width="0.254" layer="1"/>
+<via x="9" y="13.8" extent="1-16" drill="0.508"/>
+<wire x1="9" y1="13.8" x2="9" y2="15.885" width="0.254" layer="16"/>
+<wire x1="9" y1="15.885" x2="9.315" y2="16.2" width="0.254" layer="16"/>
+<wire x1="11.852" y1="9.85" x2="9" y2="12.702" width="0.254" layer="1"/>
+<wire x1="25.342915625" y1="25.2063625" x2="34.965" y2="25.2063625" width="0.254" layer="1"/>
+<via x="34.965" y="25.2063625" extent="1-16" drill="0.508"/>
 </signal>
 <signal name="GND">
@@
 <contactref element="U$2" pad="P$1"/>
 <polygon width="0.1524" layer="16">
-<vertex x="-0.05" y="0.05"/>
-<vertex x="-0.05" y="26.3"/>
-<vertex x="0.1" y="26.45"/>
+<vertex x="-0.1" y="0.05"/>
+<vertex x="-0.1" y="26.35"/>
+<vertex x="0" y="26.45"/>
 <vertex x="40.35" y="26.45"/>
 <vertex x="41.2" y="25.6"/>
