File: Hardware/Main_Controller.brd (EAGLE design)
At the start: 46.7 x 29.2 mm, 13 parts

Commit message: added capacitor to main board
Parts:
- added CSUPPLY: (no value), rcl:C1206
Connections:
- net GND: now also CSUPPLY.2
- net VCC: now also CSUPPLY.1
Routing:
- net GND: track 10.4 -> 13.7 mm, vias 4 -> 5
- net VCC: track 61.4 -> 64.3 mm
Changed lines of the file:
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@@
 </element>
 <element name="U$2" library="Personal" package="3002BATTERY" value="3002BATTERY" x="22.86" y="15.24" smashed="yes" rot="MR0"/>
+<element name="CSUPPLY" library="rcl" library_urn="urn:adsk.eagle:library:334" package="C1206" package3d_urn="urn:adsk.eagle:package:23618/2" value="" x="17.78" y="13.97" smashed="yes">
+<attribute name="NAME" x="16.51" y="15.24" size="1.27" layer="25"/>
+<attribute name="POPULARITY" value="24" x="17.78" y="13.97" size="1.778" layer="27" display="off"/>
+<attribute name="SPICEPREFIX" value="C" x="17.78" y="13.97" size="1.778" layer="27" display="off"/>
+<attribute name="VALUE" x="16.51" y="11.43" size="1.27" layer="27"/>
+</element>
 </elements>
 <signals>
@@
 <via x="19.05" y="21.59" extent="1-16" drill="0.508" diameter="0.65"/>
 <contactref element="U$2" pad="P$1"/>
+<contactref element="CSUPPLY" pad="2"/>
+<wire x1="19.18" y1="13.97" x2="17.6196" y2="12.4096" width="0.1524" layer="1"/>
+<wire x1="17.6196" y1="12.4096" x2="16.51" y2="12.4096" width="0.1524" layer="1"/>
+<via x="16.51" y="12.4096" extent="1-16" drill="0.508"/>
 </signal>
 <signal name="VCC">
@@
 <contactref element="R3" pad="2"/>
 <wire x1="15.24" y1="16.51" x2="15.24" y2="16.358" width="0.254" layer="1"/>
-<wire x1="15.24" y1="16.358" x2="11.582" y2="12.7" width="0.254" layer="1"/>
+<wire x1="15.24" y1="16.358" x2="14.046" y2="15.164" width="0.254" layer="1"/>
+<wire x1="14.046" y1="15.164" x2="11.582" y2="12.7" width="0.254" layer="1"/>
 <wire x1="21.2051" y1="16.1499" x2="15.6001" y2="16.1499" width="0.254" layer="1"/>
 <wire x1="15.6001" y1="16.1499" x2="15.24" y2="16.51" width="0.254" layer="1"/>
@@
 <wire x1="24.9346875" y1="13.0314" x2="18.7186" y2="13.0314" width="0.1524" layer="16"/>
 <wire x1="18.7186" y1="13.0314" x2="15.24" y2="16.51" width="0.1524" layer="16"/>
+<contactref element="CSUPPLY" pad="1"/>
+<wire x1="16.38" y1="13.97" x2="15.186" y2="15.164" width="0.1524" layer="1"/>
+<wire x1="15.186" y1="15.164" x2="14.046" y2="15.164" width="0.1524" layer="1"/>
 </signal>
 <signal name="RST/SBWTDIO">
