File: Hardware/Main_Controller.brd (EAGLE design)
At the start: 46.7 x 29.2 mm, 14 parts

Commit message: main board battery issue changes and cam job
Parts:
- moved R2 1.27 mm to (10.2, 20.3)
- moved R3 1.27 mm to (10.2, 25.4)
Routing:
- net VCC: track 64.3 -> 84.9 mm
Other:
- board size 46.7 x 29.2 mm -> 40 x 30 mm
