File: Hardware/Main_Controller.sch (EAGLE design)
At the start: 13 parts

Commit message: main board draft 2
Parts:
- removed BAT1: (no value), ELEC327:BATTERYBU2032SM
- added U$2: 3002BATTERY, Personal:3002BATTERY
Connections:
- net GND: now also U$2.NEG; no longer BAT1.-
- net VCC: now also U$2.POS; no longer BAT1.+
Changed lines of the file:
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@@
 <part name="P+4" library="supply1" library_urn="urn:adsk.eagle:library:371" deviceset="VCC" device=""/>
 <part name="P+5" library="supply1" library_urn="urn:adsk.eagle:library:371" deviceset="VCC" device=""/>
-<part name="BAT1" library="ELEC327" deviceset="BATTERY" device="BU2032SM"/>
 <part name="P+6" library="supply1" library_urn="urn:adsk.eagle:library:371" deviceset="VCC" device=""/>
 <part name="GND5" library="supply1" library_urn="urn:adsk.eagle:library:371" deviceset="GND" device=""/>
+<part name="U$2" library="Personal" deviceset="3002BATTERY" device=""/>
 </parts>
 <sheets>
@@
 <attribute name="VALUE" x="114.3" y="50.8" size="1.778" layer="96" rot="R90"/>
 </instance>
-<instance part="BAT1" gate="G$1" x="276.86" y="38.1" smashed="yes" rot="R270">
-<attribute name="NAME" x="281.94" y="41.91" size="1.778" layer="95" rot="R270"/>
-<attribute name="VALUE" x="270.51" y="41.91" size="1.778" layer="96" rot="R270"/>
+<instance part="P+6" gate="VCC" x="281.94" y="55.88" smashed="yes">
+<attribute name="VALUE" x="279.4" y="53.34" size="1.778" layer="96" rot="R90"/>
 </instance>
-<instance part="P+6" gate="VCC" x="276.86" y="53.34" smashed="yes">
-<attribute name="VALUE" x="274.32" y="50.8" size="1.778" layer="96" rot="R90"/>
+<instance part="GND5" gate="1" x="281.94" y="22.86" smashed="yes">
+<attribute name="VALUE" x="279.4" y="20.32" size="1.778" layer="96"/>
 </instance>
-<instance part="GND5" gate="1" x="276.86" y="25.4" smashed="yes">
-<attribute name="VALUE" x="274.32" y="22.86" size="1.778" layer="96"/>
-</instance>
+<instance part="U$2" gate="G$1" x="281.94" y="38.1" smashed="yes"/>
 </instances>
 <busses>
@@
 </segment>
 <segment>
-<pinref part="BAT1" gate="G$1" pin="-"/>
-<wire x1="276.86" y1="33.02" x2="276.86" y2="27.94" width="0.1524" layer="91"/>
+<wire x1="281.94" y1="30.48" x2="281.94" y2="25.4" width="0.1524" layer="91"/>
 <pinref part="GND5" gate="1" pin="GND"/>
+<pinref part="U$2" gate="G$1" pin="NEG"/>
 </segment>
 <segment>
@@
 </segment>
 <segment>
-<pinref part="BAT1" gate="G$1" pin="+"/>
-<wire x1="276.86" y1="43.18" x2="276.86" y2="50.8" width="0.1524" layer="91"/>
+<wire x1="281.94" y1="45.72" x2="281.94" y2="53.34" width="0.1524" layer="91"/>
 <pinref part="P+6" gate="VCC" pin="VCC"/>
+<pinref part="U$2" gate="G$1" pin="POS"/>
 </segment>
 </net>

Commit message: added capacitor to main board
Parts:
- added CSUPPLY: (no value), rcl:C-USC1206
Connections:
- net GND: now also CSUPPLY.2
- net VCC: now also CSUPPLY.1
Changed lines of the file:
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@@
 <part name="GND5" library="supply1" library_urn="urn:adsk.eagle:library:371" deviceset="GND" device=""/>
 <part name="U$2" library="Personal" deviceset="3002BATTERY" device=""/>
+<part name="CSUPPLY" library="rcl" library_urn="urn:adsk.eagle:library:334" deviceset="C-US" device="C1206" package3d_urn="urn:adsk.eagle:package:23618/2"/>
+<part name="P+7" library="supply1" library_urn="urn:adsk.eagle:library:371" deviceset="VCC" device=""/>
+<part name="GND6" library="supply1" library_urn="urn:adsk.eagle:library:371" deviceset="GND" device=""/>
 </parts>
 <sheets>
@@
 </instance>
 <instance part="U$2" gate="G$1" x="281.94" y="38.1" smashed="yes"/>
+<instance part="CSUPPLY" gate="G$1" x="299.72" y="38.1" smashed="yes">
+<attribute name="NAME" x="300.736" y="38.735" size="1.778" layer="95"/>
+<attribute name="VALUE" x="300.736" y="33.909" size="1.778" layer="96"/>
+</instance>
+<instance part="P+7" gate="VCC" x="299.72" y="48.26" smashed="yes">
+<attribute name="VALUE" x="297.18" y="45.72" size="1.778" layer="96" rot="R90"/>
+</instance>
+<instance part="GND6" gate="1" x="299.72" y="25.4" smashed="yes">
+<attribute name="VALUE" x="297.18" y="22.86" size="1.778" layer="96"/>
+</instance>
 </instances>
 <busses>
@@
 <label x="15.24" y="20.32" size="1.778" layer="95"/>
 </segment>
+<segment>
+<pinref part="GND6" gate="1" pin="GND"/>
+<pinref part="CSUPPLY" gate="G$1" pin="2"/>
+<wire x1="299.72" y1="27.94" x2="299.72" y2="33.02" width="0.1524" layer="91"/>
+</segment>
 </net>
 <net name="VCC" class="0">
@@
 <pinref part="U$2" gate="G$1" pin="POS"/>
 </segment>
+<segment>
+<pinref part="CSUPPLY" gate="G$1" pin="1"/>
+<pinref part="P+7" gate="VCC" pin="VCC"/>
+<wire x1="299.72" y1="40.64" x2="299.72" y2="45.72" width="0.1524" layer="91"/>
+</segment>
 </net>
